Commit message: wip: use different colours for pioneers 1 and 2

File: p3dx_description/urdf/p3dx/pioneer3dx_body.xacro (robot description, xacro)
@@ -13,5 +13,5 @@
     <link name="${parent}"/>
     <!-- Chassis -->
-    <xacro:pioneer_chassis name="${name}" parent="base_link" xyz="0 0 0" rpy="0 0 0"  meshes="${meshes}"/>
+    <xacro:pioneer_chassis name="${name}" parent="base_link" xyz="0 0 0" rpy="0 0 0"  meshes="${meshes}" robot_namespace="${robot_namespace}"/>
     <!-- Front Sonar -->
     <xacro:pioneer_sonar name="sonar" parent="${name}" xyz="0.109 0 0.209" rpy="0 0 0"  meshes="${meshes}"/>

File: p3dx_description/urdf/p3dx/pioneer3dx_chassis.xacro (robot description, xacro)
@@ -2,5 +2,5 @@
 <robot xmlns:xacro="http://ros.org/wiki/xacro">
   <xacro:property name="M_PI" value="3.1415926535897931" />
-  <xacro:macro name="pioneer_chassis" params="name parent xyz rpy meshes">
+  <xacro:macro name="pioneer_chassis" params="name parent xyz rpy meshes robot_namespace">
   <!-- Chassis -->
   <joint name="${parent}_${name}_joint" type="fixed">
@@ -42,7 +42,19 @@
         <mesh filename="${meshes}/top.stl"/>
       </geometry>
-      <material name="TopBlack">
-        <color rgba="0.038 0.038 0.038 1.0"/>
-      </material>
+      <xacro:if value="${robot_namespace == 'pioneer1'}">
+        <material name="TopGreen">
+          <color rgba="0.0 0.8 0.0 1.0"/>
+        </material>
+      </xacro:if>
+      <xacro:if value="${robot_namespace == 'pioneer2'}">
+        <material name="TopRed">
+          <color rgba="0.8 0.0 0.0 1.0"/>
+        </material>
+      </xacro:if>
+      <xacro:if value="${robot_namespace == '/'}">
+        <material name="TopBlack">
+          <color rgba="0.038 0.038 0.038 1.0"/>
+        </material>
+      </xacro:if>
     </visual>
     <collision>
